Commit message: ri4のモデルに胴体の表示を成功させた。次回は、右鼠径部の表示である。

File: urdf/er14000w.urdf (robot description, URDF)
Before this commit: robot ri4, 8 links, 7 joints
Links:
- link body: geometry collision box size=0.2 0.1 0.5; visual box size=0.2 0.1 0.5

Commit message: 鼠径部完了。次回、太もも

File: urdf/er14000w.urdf (robot description, URDF)
Before this commit: robot ri4, 8 links, 7 joints
Links:
- link link1: geometry collision box size=0.2 0.05 0.1; visual box size=0.2 0.05 0.1
Joints:
- joint joint1: origin xyz=0 0 0.3 rpy=0 0 0 -> xyz=0.1 0 0.0 rpy=0 0 0

Commit message: 太腿完成。次回、スネ。

File: urdf/er14000w.urdf (robot description, URDF)
Before this commit: robot ri4, 8 links, 7 joints
Links:
- link link2: geometry collision box size=0.1 0.02 0.4; visual box size=0.1 0.02 0.4
Joints:
- joint joint2: origin xyz=0 0 0.5 rpy=0 0 0 -> xyz=0.1 0 -0.1 rpy=0 0 0

Commit message: スネ完了。次回、踝。問題：膝関節がcpp指定通り動いていない。問題持ち越し。

File: urdf/er14000w.urdf (robot description, URDF)
Before this commit: robot ri4, 8 links, 7 joints
Links:
- link link3: geometry collision box size=0.1 0.01 0.4; visual box size=0.1 0.01 0.4
Joints:
- joint joint3: axis 0 0 1 -> 1 0 0; origin xyz=0 0 0.5 rpy=0 0 0 -> xyz=0 0 -0.4 rpy=0 0 3.1415

Commit message: 右踝完了。次回、踝下。

File: urdf/er14000w.urdf (robot description, URDF)
Before this commit: robot ri4, 8 links, 7 joints
Links:
- link linkx: geometry collision box size=0.2 0.05 0.1; visual box size=0.2 0.05 0.1
Joints:
- joint joint0: origin xyz=1 1 1 rpy=0 0 0 -> xyz=1 1 1.2 rpy=0 0 0
- joint jointx: origin xyz=0.4 0 0.3 rpy=0 0 0 -> xyz=0 0 -0.4 rpy=0 0 3.1415926; parent body -> link3

Commit message: 右踝下完了。次回、左鼠径部。方針：取り敢えずurdfの形状優先。運動はcppのとき追記。

File: urdf/er14000w.urdf (robot description, URDF)
Before this commit: robot ri4, 8 links, 7 joints
Links:
- link linkx2: geometry collision box size=0.2 0.3 0.01; visual box size=0.2 0.3 0.01
Joints:
- joint jointx2: axis (none) -> 0 1 0; origin xyz=0.4 0 0 rpy=0 0 0 -> xyz=0 0 -0.1 rpy=0 0 0

Commit message: 左鼠径部完了。ri4の構成要素使い切る。次回：名称整理。

File: urdf/er14000w.urdf (robot description, URDF)
Before this commit: robot ri4, 8 links, 7 joints
Links:
- link linky: geometry collision box size=0.2 0.05 0.1; visual box size=0.2 0.05 0.1
Joints:
- joint jointy: axis 0 1 0 -> 0 -1 0; origin xyz=0 0.2 0.3 rpy=0 0 0 -> xyz=-0.1 0 0.0 rpy=0 0 0

Commit message: Link名の変更完了。次回、Jointm名の変更。

File: urdf/er14000w.urdf (robot description, URDF)
Before this commit: robot ri4, 8 links, 7 joints
Links:
- removed link body
- removed link link1
- removed link link2
- removed link link3
- removed link linkx
- removed link linkx2
- removed link linky
- added link body1, mass 20; collision box size=0.2 0.1 0.5; visual box size=0.2 0.1 0.5
- added link body2, mass 0.1; collision box size=0.2 0.05 0.1; visual box size=0.2 0.05 0.1
- added link body3, mass 0.1; collision box size=0.1 0.02 0.4; visual box size=0.1 0.02 0.4
- added link body4, mass 0.1; collision box size=0.1 0.01 0.4; visual box size=0.1 0.01 0.4
- added link body5, mass 0.1; collision box size=0.2 0.05 0.1; visual box size=0.2 0.05 0.1
- added link body6, mass 0.1; collision box size=0.2 0.3 0.01; visual box size=0.2 0.3 0.01
- added link body7, mass 0.1; collision box size=0.2 0.05 0.1; visual box size=0.2 0.05 0.1
Joints:
- joint joint0: child body -> body1; origin xyz=1 1 1.2 rpy=0 0 0 -> xyz=1 1 1.1 rpy=0 0 0
- joint joint1: child link1 -> body2; parent body -> body1
- joint joint2: child link2 -> body3; parent link1 -> body2
- joint joint3: child link3 -> body4; parent link2 -> body3
- joint jointx: child linkx -> body5; parent link3 -> body4
- joint jointx2: child linkx2 -> body6; parent linkx -> body5
- joint jointy: child linky -> body7; parent body -> body1

Commit message: 腕以外のモデル完成。シミュレーションは、これでやっていく。次回：コードの整理

File: urdf/er14000w.urdf (robot description, URDF)
Before this commit: robot ri4, 8 links, 7 joints
Links:
- added link body10, mass 0.1; collision box size=0.2 0.05 0.1; visual box size=0.2 0.05 0.1
- added link body11, mass 0.1; collision box size=0.2 0.3 0.01; visual box size=0.2 0.3 0.01
- added link body8, mass 0.1; collision box size=0.1 0.02 0.4; visual box size=0.1 0.02 0.4
- added link body9, mass 0.1; collision box size=0.1 0.01 0.4; visual box size=0.1 0.01 0.4
Joints:
- added joint joint22: type revolute, parent body7, child body8, origin xyz=-0.1 0 -0.1 rpy=0 0 0, axis 1 0 0, limit lower=-2.617 upper=2.617 effort=30 velocity=1.571
- added joint joint23: type revolute, parent body8, child body9, origin xyz=0 0 -0.4 rpy=0 0 3.1415, axis 1 0 0, limit lower=-2.617 upper=2.617 effort=30 velocity=1.571
- added joint joint2x: type revolute, parent body9, child body10, origin xyz=0 0 -0.4 rpy=0 0 3.1415926, axis 1 0 0, limit lower=-2.617 upper=2.617 effort=30 velocity=1.571
- added joint joint2x2: type fixed, parent body10, child body11, origin xyz=0 0 -0.1 rpy=0 0 0, axis 0 1 0

Commit message: モータ番号の整理、モデルに色をつけるが完了。次回、制御を行う。

File: urdf/er14000w.urdf (robot description, URDF)
Before this commit: robot ri4, 12 links, 11 joints
Links:
- link body10: geometry visual box size=0.2 0.05 0.1
- link body5: geometry visual box size=0.2 0.05 0.1
Joints:
- removed joint joint22
- removed joint joint23
- removed joint joint2x
- removed joint joint2x2
- removed joint jointx
- removed joint jointx2
- removed joint jointy
- added joint joint10: type revolute, parent body10, child body11, origin xyz=0 0 -0.1 rpy=0 0 0, axis 0 1 0, limit lower=-2.617 upper=2.617 effort=30 velocity=1.571
- added joint joint4: type revolute, parent body4, child body5, origin xyz=0 0 -0.4 rpy=0 0 3.1415926, axis 1 0 0, limit lower=-2.617 upper=2.617 effort=30 velocity=1.571
- added joint joint5: type revolute, parent body5, child body6, origin xyz=0 0 -0.1 rpy=0 0 0, axis 0 1 0, limit lower=-2.617 upper=2.617 effort=30 velocity=1.571
- added joint joint6: type revolute, parent body1, child body7, origin xyz=-0.1 0 0.0 rpy=0 0 0, axis 0 -1 0, limit lower=-2.617 upper=2.617 effort=30 velocity=1.571
- added joint joint7: type revolute, parent body7, child body8, origin xyz=-0.1 0 -0.1 rpy=0 0 0, axis 1 0 0, limit lower=-2.617 upper=2.617 effort=30 velocity=1.571
- added joint joint8: type revolute, parent body8, child body9, origin xyz=0 0 -0.4 rpy=0 0 3.1415, axis 1 0 0, limit lower=-2.617 upper=2.617 effort=30 velocity=1.571
- added joint joint9: type revolute, parent body9, child body10, origin xyz=0 0 -0.4 rpy=0 0 3.1415926, axis 1 0 0, limit lower=-2.617 upper=2.617 effort=30 velocity=1.571

Commit message: 腕の設置OK。関節は全てfix。次回：足の運動が観察可能な腕に形状変更。

File: urdf/er14000w.urdf (robot description, URDF)
Before this commit: robot ri4, 12 links, 11 joints
Links:
- added link body12; visual box size=0.2 0.05 0.1
- added link body13; visual box size=0.1 0.02 0.3
- added link body14; visual box size=0.1 0.01 0.3
- added link body15; visual box size=0.2 0.05 0.1
- added link body16; visual box size=0.1 0.02 0.3
- added link body17; visual box size=0.1 0.01 0.3
Joints:
- added joint joint11: type fixed, parent body1, child body12, origin xyz=0.1 0 0.5 rpy=0 0 0, axis 0 1 0
- added joint joint12: type fixed, parent body12, child body13, origin xyz=0.1 0 -0.1 rpy=0 0 0
- added joint joint13: type fixed, parent body13, child body14, origin xyz=0 0 -0.3 rpy=0 0 0
- added joint joint14: type fixed, parent body1, child body15, origin xyz=-0.1 0 0.5 rpy=0 0 0, axis 0 1 0
- added joint joint15: type fixed, parent body15, child body16, origin xyz=-0.1 0 -0.1 rpy=0 0 3.1415
- added joint joint16: type fixed, parent body16, child body17, origin xyz=0 0 -0.3 rpy=0 0 0, limit lower=-1.5 upper=1.5 effort=0 velocity=0

Commit message: 足の動きを見るためのモデル完成。次回：左右の股関節y軸の設定を比較し、統一。 左は振り子、右は固定。右は制御できている。左は制御無し。確認を行う。

File: urdf/er14000w.urdf (robot description, URDF)
Before this commit: robot ri4, 18 links, 17 joints
Links:
- link body12: geometry visual box size=0.3 0.05 0.1
- link body13: geometry visual box size=0.1 0.02 1.4
- link body14: geometry collision box size=0.1 0.3 0.1; visual box size=0.1 0.3 0.1
- link body15: geometry visual box size=0.3 0.05 0.1
- link body16: geometry visual box size=0.1 0.02 1.4
- link body17: geometry collision box size=0.1 0.3 0.1; visual box size=0.1 0.3 0.1
Joints:
- joint joint0: origin xyz=1 1 1.1 rpy=0 0 0 -> xyz=1 1 1.2 rpy=0 0 0
- joint joint12: origin xyz=0.1 0 -0.1 rpy=0 0 0 -> xyz=0.3 0 -0.1 rpy=0 0 0
- joint joint13: origin xyz=0 0 -0.3 rpy=0 0 0 -> xyz=0 0 -1.4 rpy=0 0 0
- joint joint15: origin xyz=-0.1 0 -0.1 rpy=0 0 3.1415 -> xyz=-0.3 0 -0.1 rpy=0 0 3.1415
- joint joint16: limit lower=-1.5 upper=1.5 effort=0 velocity=0 -> (none); origin xyz=0 0 -0.3 rpy=0 0 0 -> xyz=0 0 -1.4 rpy=0 0 0

Commit message: 左右の股関節が違うところを修正。次回：制御をいじって見る。

File: urdf/er14000w.urdf (robot description, URDF)
Before this commit: robot ri4, 18 links, 17 joints
Joints:
- joint joint6: axis 0 -1 0 -> 0 1 0

Commit message: 左足の動きは、修正完了。次回：腕を短くして、実際の歩行を行う。rvizは取り敢えず断念。 結果として、rvizの動きとgazeboの動きは、一致した。

File: urdf/er14000w.urdf (robot description, URDF)
Before this commit: robot ri4, 18 links, 17 joints
Joints:
- joint joint10: axis 0 1 0 -> 0 -1 0
- joint joint6: axis 0 1 0 -> 0 -1 0

Commit message: 腕を短くした。歩行開始のプログラムを起動うると、転倒。転倒防止の前に。運動データの確認 運動データの軸回転方向の確認を行う。本来あるべき方向と違うと思われるのは、左鼠径部Yと左踝Yである。 両軸ともにマイナスが付加されているが、本来は必要ない。 このマイナスを外すために、データの見直しを行う。

File: urdf/er14000w.urdf (robot description, URDF)
Before this commit: robot ri4, 18 links, 17 joints
Links:
- link body13: geometry visual box size=0.1 0.02 0.3
- link body14: geometry visual box size=0.1 0.1 0.3
- link body16: geometry visual box size=0.1 0.02 0.3
- link body17: geometry visual box size=0.1 0.1 0.3
Joints:
- joint joint0: origin xyz=1 1 1.2 rpy=0 0 0 -> xyz=1 1 1.05 rpy=0 0 0
- joint joint13: origin xyz=0 0 -1.4 rpy=0 0 0 -> xyz=0 0 -.3 rpy=0 0 0
- joint joint16: origin xyz=0 0 -1.4 rpy=0 0 0 -> xyz=0 0 -0.3 rpy=0 0 0

Commit message: urdfの左股関節と踝のY肉について、不要なマイナスを削除。伴いcppを修正。次回：直立から歩行始めの姿勢変更

File: urdf/er14000w.urdf (robot description, URDF)
Before this commit: robot ri4, 18 links, 17 joints
Joints:
- joint joint10: axis 0 -1 0 -> 0 1 0
- joint joint6: axis 0 -1 0 -> 0 1 0

Commit message: 補間OK：補助の腕をつけて足の動きを確認。次回、モータの出力を上げて歩行を安定化

File: urdf/er14000w.urdf (robot description, URDF)
Before this commit: robot ri4, 18 links, 17 joints
Links:
- link body13: geometry visual box size=0.1 0.02 1.3
- link body14: geometry collision box size=0.1 1.2 0.1; visual box size=0.1 1.2 0.1
- link body16: geometry visual box size=0.1 0.02 1.3
- link body17: geometry collision box size=0.1 1.2 0.1; visual box size=0.1 1.2 0.1
Joints:
- joint joint11: origin xyz=0.1 0 0.5 rpy=0 0 0 -> xyz=0.1 0 0.5 rpy=0 -0.23 0
- joint joint13: origin xyz=0 0 -.3 rpy=0 0 0 -> xyz=0 0 -1.3 rpy=0 0 0
- joint joint14: origin xyz=-0.1 0 0.5 rpy=0 0 0 -> xyz=-0.1 0 0.5 rpy=0 0.23 0
- joint joint16: origin xyz=0 0 -0.3 rpy=0 0 0 -> xyz=0 0 -1.3 rpy=0 0 0

Commit message: GazeboシミュレーションによるRBの歩行完了。次回：腕を戻す。ただし、また補助として使うので、コメントアウト。今後：マクロで定義してある定数をパラメータに変更していく。

File: urdf/er14000w.urdf (robot description, URDF)
Before this commit: robot ri4, 18 links, 17 joints
Links:
- link body1: mass 20 -> 5
Joints:
- joint joint1: limit lower=-2.617 upper=2.617 effort=30 velocity=1.571 -> lower=-2.617 upper=2.617 effort=360 velocity=1.571
- joint joint10: limit lower=-2.617 upper=2.617 effort=30 velocity=1.571 -> lower=-2.617 upper=2.617 effort=360 velocity=1.571
- joint joint11: origin xyz=0.1 0 0.5 rpy=0 -0.23 0 -> xyz=0.1 0 0.5 rpy=0 -0.54 0
- joint joint14: origin xyz=-0.1 0 0.5 rpy=0 0.23 0 -> xyz=-0.1 0 0.5 rpy=0 0.54 0
- joint joint2: limit lower=-2.617 upper=2.617 effort=30 velocity=1.571 -> lower=-2.617 upper=2.617 effort=360 velocity=1.571
- joint joint3: limit lower=-2.617 upper=2.617 effort=30 velocity=1.571 -> lower=-2.617 upper=2.617 effort=360 velocity=1.571
- joint joint4: limit lower=-2.617 upper=2.617 effort=30 velocity=1.571 -> lower=-2.617 upper=2.617 effort=360 velocity=1.571
- joint joint5: limit lower=-2.617 upper=2.617 effort=30 velocity=1.571 -> lower=-2.617 upper=2.617 effort=360 velocity=1.571
- joint joint6: limit lower=-2.617 upper=2.617 effort=30 velocity=1.571 -> lower=-2.617 upper=2.617 effort=360 velocity=1.571
- joint joint7: limit lower=-2.617 upper=2.617 effort=30 velocity=1.571 -> lower=-2.617 upper=2.617 effort=360 velocity=1.571
- joint joint8: limit lower=-2.617 upper=2.617 effort=30 velocity=1.571 -> lower=-2.617 upper=2.617 effort=360 velocity=1.571
- joint joint9: limit lower=-2.617 upper=2.617 effort=30 velocity=1.571 -> lower=-2.617 upper=2.617 effort=360 velocity=1.571

Commit message: Webに歩行運動のgifをアップ。歩行が不安定である。機体の形状によるものと思われる。次回、細いロボットを作ってみる。 細いロボットを作ることでえ、機体の形状とシミュレーションの影響を確認する。

File: urdf/er14000w.urdf (robot description, URDF)
Before this commit: robot ri4, 18 links, 17 joints
Links:
- link body13: geometry visual box size=0.1 0.02 0.3
- link body14: geometry visual box size=0.1 0.1 0.3
- link body16: geometry visual box size=0.1 0.02 0.3
- link body17: geometry visual box size=0.1 0.1 0.3
Joints:
- joint joint13: origin xyz=0 0 -1.3 rpy=0 0 0 -> xyz=0 0 -.3 rpy=0 0 0
- joint joint16: origin xyz=0 0 -1.3 rpy=0 0 0 -> xyz=0 0 -0.3 rpy=0 0 0

Commit message: 構成部材の形状と強度には、因果関係なし。chatGPTにも確認したが、強度を定義するパラメータは無し。 不安定の原因は、モータトルクと考えられる。次回、さらなるトルクアップを行って見る。

File: urdf/er14000w.urdf (robot description, URDF)
Before this commit: robot ri4, 18 links, 17 joints
Links:
- link body6: geometry collision box size=0.2 0.3 0.01; visual box size=0.2 0.3 0.0001
